File: hw/boards/tk1/application_fpga.kicad_sch (KiCad schematic)
At the start: 38 parts, among them U6 ICE40UP5K-SG48ITR, U8 W25Q80DVUXIE

Commit message: Replaced Cap w. spring contacts
Parts:
- added U11: (no value), symbol mta1:1674954-1
- C8: value 1uF -> (none); footprint Capacitor_SMD:C_1206_3216Metric -> (none); now left out of the parts list
- U10: value (none) -> PT2043AT6; footprint (none) -> Package_TO_SOT_SMD:SOT-23-6
Connections:
- net TOUCH_PAD: now also U11.1
Other:
- note added: "Note: C8 Not populated. U11 used instead but on C8 footprint."
